Commit message: right wheel

File: go-chase-it/catkin_ws/src/my_robot/urdf/my_robot.xacro (robot description, xacro)
@@ -10,4 +10,12 @@
     <origin xyz="0 0.15 0" rpy="0 0 0"/>
     <child link="left_wheel"/>
+    <parent link="chassis"/>
+    <axis xyz="0 1 0" rpy="0 0 0"/>
+    <limit effort="10000" velocity="1000"/>
+    <dynamics damping="1.0" friction="1.0"/>
+  </joint>
+<joint type="continuous" name="right_wheel_hinge">
+    <origin xyz="0 -0.15 0" rpy="0 0 0"/>
+    <child link="right_wheel"/>
     <parent link="chassis"/>
     <axis xyz="0 1 0" rpy="0 0 0"/>
@@ -67,5 +75,5 @@
     <inertial>
       <mass value="5.0"/>
-      <origin xyz="0 0 0" rpy=" 0 1.5707 1.5707"/>
+      <origin xyz="0 0 0" rpy="0 1.5707 1.5707"/>
       <inertia
           ixx="0.1" ixy="0" ixz="0"
@@ -75,5 +83,5 @@
     </inertial>
     <collision name='left_wheel_collision'>
-      <origin xyz="0 0 0" rpy=" 0 1.5707 1.5707"/>
+      <origin xyz="0 0 0" rpy="0 1.5707 1.5707"/>
       <geometry>
         <cylinder radius="0.1" length="0.05"/>
@@ -81,5 +89,29 @@
     </collision>
     <visual name='left_wheel_visual'>
-      <origin xyz="0 0 0" rpy=" 0 1.5707 1.5707"/>
+      <origin xyz="0 0 0" rpy="0 1.5707 1.5707"/>
+      <geometry>
+        <cylinder radius="0.1" length="0.05"/>
+      </geometry>
+    </visual>
+  </link>
+  <!-- Right wheel -->
+  <link name="right_wheel">
+    <inertial>
+      <mass value="5.0"/>
+      <origin xyz="0 0 0" rpy="0 1.5707 1.5707"/>
+      <inertia
+          ixx="0.1" ixy="0" ixz="0"
+          iyy="0.1" iyz="0"
+          izz="0.1"
+      />
+    </inertial>
+    <collision name='right_wheel_collision'>
+      <origin xyz="0 0 0" rpy="0 1.5707 1.5707"/>
+      <geometry>
+        <cylinder radius="0.1" length="0.05"/>
+      </geometry>
+    </collision>
+    <visual name='right_wheel_visual'>
+      <origin xyz="0 0 0" rpy="0 1.5707 1.5707"/>
       <geometry>
         <cylinder radius="0.1" length="0.05"/>

Commit message: camera

File: go-chase-it/catkin_ws/src/my_robot/urdf/my_robot.xacro (robot description, xacro)
@@ -15,5 +15,5 @@
     <dynamics damping="1.0" friction="1.0"/>
   </joint>
-<joint type="continuous" name="right_wheel_hinge">
+  <joint type="continuous" name="right_wheel_hinge">
     <origin xyz="0 -0.15 0" rpy="0 0 0"/>
     <child link="right_wheel"/>
@@ -22,4 +22,10 @@
     <limit effort="10000" velocity="1000"/>
     <dynamics damping="1.0" friction="1.0"/>
+  </joint>
+  <joint type="fixed" name="camera_joint">
+    <origin xyz="0.2 0 0" rpy="0 0 0"/>
+    <child link="camera"/>
+    <parent link="chassis"/>
+    <axis xyz="0 1 0" rpy="0 0 0"/>
   </joint>
   <link name='chassis'>
@@ -119,3 +125,23 @@
     </visual>
   </link>
+  <!-- Camera -->
+  <link name="camera">
+    <inertial>
+      <mass value="0.1"/>
+      <origin xyz="0 0 0" rpy="0 0 0"/>
+      <inertia ixx="1e-6" ixy="0" ixz="0" iyy="1e-6" iyz="0" izz="1e-6"/>
+    </inertial>
+    <collision name='camera_collision'>
+      <origin xyz="0 0 0" rpy="0 0 0"/>
+      <geometry>
+        <box size="0.05 0.05 0.05"/>
+      </geometry>
+    </collision>
+    <visual name='camera_visual'>
+      <origin xyz="0 0 0" rpy="0 0 0"/>
+      <geometry>
+        <box size="0.05 0.05 0.05"/>
+      </geometry>
+    </visual>
+  </link>
 </robot>

Commit message: finishing model

File: go-chase-it/catkin_ws/src/my_robot/urdf/my_robot.xacro (robot description, xacro)
@@ -29,4 +29,10 @@
     <axis xyz="0 1 0" rpy="0 0 0"/>
   </joint>
+ <joint type="fixed" name="hokuyo_joint">
+    <origin xyz="0.15 0.1 0" rpy="0 0 0"/>
+    <child link="hokuyo"/>
+    <parent link="chassis"/>
+    <axis xyz="0 1 0" rpy="0 0 0"/>
+  </joint>
   <link name='chassis'>
     <pose>0 0 0.1 0 0 0</pose>
@@ -51,4 +57,7 @@
         <box size=".4 .2 .1"/>
       </geometry>
+      <material>
+        <color rgba="0.2 0.9 0.2 1" />
+      </material>
     </visual>
     <collision name='back_caster_collision'>
@@ -99,4 +108,7 @@
         <cylinder radius="0.1" length="0.05"/>
       </geometry>
+      <material>
+        <color rgba="0.2 0.2 0.9 1" />
+      </material>
     </visual>
   </link>
@@ -123,4 +135,7 @@
         <cylinder radius="0.1" length="0.05"/>
       </geometry>
+      <material>
+        <color rgba="0.2 0.2 0.9 1" />
+      </material>
     </visual>
   </link>
@@ -143,4 +158,27 @@
         <box size="0.05 0.05 0.05"/>
       </geometry>
+      <material>
+        <color rgba="0.8 0.2 0.8 1" />
+      </material>
+    </visual>
+  </link>
+  <!-- Lidar -->
+  <link name="hokuyo">
+    <inertial>
+      <mass value="1e-5"/>
+      <origin xyz="0 0 0" rpy="0 0 0"/>
+      <inertia ixx="1e-6" ixy="0" ixz="0" iyy="1e-6" iyz="0" izz="1e-6"/>
+    </inertial>
+    <collision name='hokuyo_collision'>
+      <origin xyz="0 0 0" rpy="0 0 0"/>
+      <geometry>
+        <box size="0.1 0.1 0.1"/>
+      </geometry>
+    </collision>
+    <visual name='hokuyo_visual'>
+      <origin xyz="0 0 0" rpy="0 0 0"/>
+      <geometry>
+        <mesh filename="package://my_robot/meshes/hokuyo.dae"/>
+      </geometry>
     </visual>
   </link>

Commit message: coords fix

File: go-chase-it/catkin_ws/src/my_robot/urdf/my_robot.xacro (robot description, xacro)
@@ -29,6 +29,6 @@
     <axis xyz="0 1 0" rpy="0 0 0"/>
   </joint>
- <joint type="fixed" name="hokuyo_joint">
-    <origin xyz="0.15 0.1 0" rpy="0 0 0"/>
+  <joint type="fixed" name="hokuyo_joint">
+    <origin xyz="0.15 0 .1" rpy="0 0 0"/>
     <child link="hokuyo"/>
     <parent link="chassis"/>

Commit message: materials

File: go-chase-it/catkin_ws/src/my_robot/urdf/my_robot.xacro (robot description, xacro)
@@ -1,4 +1,16 @@
 <?xml version='1.0'?>
 <robot name="my_robot" xmlns:xacro="http://www.ros.org/wiki/xacro">
+  <material name="green">
+    <color rgba="0.2 0.9 0.2 1" />
+  </material>
+  <material name="blue">
+    <color rgba="0.2 0.2 0.9 1" />
+  </material>
+  <material name="red">
+    <color rgba="0.9 0.2 0.2 1" />
+  </material>
+  <material name="yellow">
+    <color rgba="0.8 0.8 0.2 1" />
+  </material>
   <link name="robot_footprint"></link>
   <joint name="robot_footprint_joint" type="fixed">
@@ -57,7 +69,5 @@
         <box size=".4 .2 .1"/>
       </geometry>
-      <material>
-        <color rgba="0.2 0.9 0.2 1" />
-      </material>
+      <material name="green"/>
     </visual>
     <collision name='back_caster_collision'>
@@ -72,4 +82,5 @@
         <sphere radius="0.05"/>
       </geometry>
+      <material name="green"/>
     </visual>
     <collision name='front_caster_collision'>
@@ -84,4 +95,5 @@
         <sphere radius="0.05"/>
       </geometry>
+      <material name="green"/>
     </visual>
   </link>
@@ -108,7 +120,5 @@
         <cylinder radius="0.1" length="0.05"/>
       </geometry>
-      <material>
-        <color rgba="0.2 0.2 0.9 1" />
-      </material>
+      <material name="blue"/>
     </visual>
   </link>
@@ -135,7 +145,5 @@
         <cylinder radius="0.1" length="0.05"/>
       </geometry>
-      <material>
-        <color rgba="0.2 0.2 0.9 1" />
-      </material>
+      <material name="blue"/>
     </visual>
   </link>
@@ -158,7 +166,5 @@
         <box size="0.05 0.05 0.05"/>
       </geometry>
-      <material>
-        <color rgba="0.8 0.2 0.8 1" />
-      </material>
+      <material name="red"/>
     </visual>
   </link>

Commit message: materials

File: go-chase-it/catkin_ws/src/my_robot/urdf/my_robot.xacro (robot description, xacro)
@@ -2,16 +2,4 @@
 <robot name="my_robot" xmlns:xacro="http://www.ros.org/wiki/xacro">
   <xacro:include filename="$(find my_robot)/urdf/my_robot.gazebo" />
-  <material name="green">
-    <color rgba="0.2 0.9 0.2 1" />
-  </material>
-  <material name="blue">
-    <color rgba="0.2 0.2 0.9 1" />
-  </material>
-  <material name="red">
-    <color rgba="0.9 0.2 0.2 1" />
-  </material>
-  <material name="yellow">
-    <color rgba="0.8 0.8 0.2 1" />
-  </material>
   <link name="robot_footprint"></link>
   <joint name="robot_footprint_joint" type="fixed">
@@ -70,5 +58,4 @@
         <box size=".4 .2 .1"/>
       </geometry>
-      <material name="green"/>
     </visual>
     <collision name='back_caster_collision'>
@@ -83,5 +70,4 @@
         <sphere radius="0.05"/>
       </geometry>
-      <material name="green"/>
     </visual>
     <collision name='front_caster_collision'>
@@ -96,5 +82,4 @@
         <sphere radius="0.05"/>
       </geometry>
-      <material name="green"/>
     </visual>
   </link>
@@ -121,5 +106,4 @@
         <cylinder radius="0.1" length="0.05"/>
       </geometry>
-      <material name="blue"/>
     </visual>
   </link>
@@ -146,5 +130,4 @@
         <cylinder radius="0.1" length="0.05"/>
       </geometry>
-      <material name="blue"/>
     </visual>
   </link>
@@ -167,5 +150,4 @@
         <box size="0.05 0.05 0.05"/>
       </geometry>
-      <material name="red"/>
     </visual>
   </link>

Commit message: robot size modification

File: go-chase-it/catkin_ws/src/my_robot/urdf/my_robot.xacro (robot description, xacro)
@@ -25,5 +25,5 @@
   </joint>
   <joint type="fixed" name="camera_joint">
-    <origin xyz="0.2 0 0" rpy="0 0 0"/>
+    <origin xyz="0.25 0 0" rpy="0 0 0"/>
     <child link="camera"/>
     <parent link="chassis"/>
@@ -50,5 +50,5 @@
       <origin xyz="0 0 0" rpy=" 0 0 0"/>
       <geometry>
-        <box size=".4 .2 .1"/>
+        <box size=".5 .2 .1"/>
       </geometry>
     </collision>
@@ -56,5 +56,5 @@
       <origin xyz="0 0 0" rpy=" 0 0 0"/>
       <geometry>
-        <box size=".4 .2 .1"/>
+        <box size=".5 .2 .1"/>
       </geometry>
     </visual>
@@ -98,5 +98,5 @@
       <origin xyz="0 0 0" rpy="0 1.5707 1.5707"/>
       <geometry>
-        <cylinder radius="0.1" length="0.05"/>
+        <cylinder radius="0.1" length="0.04"/>
       </geometry>
     </collision>
@@ -104,5 +104,5 @@
       <origin xyz="0 0 0" rpy="0 1.5707 1.5707"/>
       <geometry>
-        <cylinder radius="0.1" length="0.05"/>
+        <cylinder radius="0.1" length="0.04"/>
       </geometry>
     </visual>
@@ -122,5 +122,5 @@
       <origin xyz="0 0 0" rpy="0 1.5707 1.5707"/>
       <geometry>
-        <cylinder radius="0.1" length="0.05"/>
+        <cylinder radius="0.1" length="0.04"/>
       </geometry>
     </collision>
@@ -128,5 +128,5 @@
       <origin xyz="0 0 0" rpy="0 1.5707 1.5707"/>
       <geometry>
-        <cylinder radius="0.1" length="0.05"/>
+        <cylinder radius="0.1" length="0.04"/>
       </geometry>
     </visual>
